File: PiPhoneV0.kicad_sch (KiCad schematic)
At the start: 44 parts, among them IC1 LM386M-1_NOPB, J1 GPIO, SW1 SW_Push, SW10 SW_Push, SW11 SW_Push, SW12 SW_Push, SW13 SW_Push, SW14 SW_Push, SW15 SW_Push, SW16 SW_Push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

Commit message: chore: body curve
Parts:
- C1, C4: footprint Capacitor_THT:CP_Axial_L10.0mm_D4.5mm_P15.00mm_Horizontal -> Capacitor_SMD:CP_Elec_3x5.3
- C2, C3: footprint Capacitor_THT:CP_Axial_L10.0mm_D4.5mm_P15.00mm_Horizontal -> Capacitor_SMD:C_0201_0603Metric
- D1, D10, D11, D12, D13, D14, D15, D16, D17, D18, D2, D3, D4, D5, D6, D7, D8, D9: footprint Diode_THT:D_5KPW_P12.70mm_Horizontal -> Diode_SMD:D_0201_0603Metric
- R3: footprint Resistor_SMD:R_0201_0603Metric -> Diode_SMD:D_0201_0603Metric
Changed lines of the file:
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@@
 			)
 		)
-		(property "Footprint" "Capacitor_THT:CP_Axial_L10.0mm_D4.5mm_P15.00mm_Horizontal"
+		(property "Footprint" "Capacitor_SMD:CP_Elec_3x5.3"
 			(at 109.22 101.6 0)
 			(effects
@@
 			)
 		)
-		(property "Footprint" "Diode_THT:D_5KPW_P12.70mm_Horizontal"
+		(property "Footprint" "Diode_SMD:D_0201_0603Metric"
 			(at 205.74 102.87 0)
 			(effects
@@
 			)
 		)
-		(property "Footprint" "Diode_THT:D_5KPW_P12.70mm_Horizontal"
+		(property "Footprint" "Diode_SMD:D_0201_0603Metric"
 			(at 205.74 91.44 0)
 			(effects
@@
 			)
 		)
-		(property "Footprint" "Diode_THT:D_5KPW_P12.70mm_Horizontal"
+		(property "Footprint" "Diode_SMD:D_0201_0603Metric"
 			(at 205.74 68.58 0)
 			(effects
@@
 			)
 		)
-		(property "Footprint" "Diode_THT:D_5KPW_P12.70mm_Horizontal"
+		(property "Footprint" "Diode_SMD:D_0201_0603Metric"
 			(at 205.74 80.01 0)
 			(effects
@@
 			)
 		)
-		(property "Footprint" "Resistor_SMD:R_0201_0603Metric"
+		(property "Footprint" "Diode_SMD:D_0201_0603Metric"
 			(at 66.548 121.92 90)
 			(effects
@@
 			)
 		)
-		(property "Footprint" "Diode_THT:D_5KPW_P12.70mm_Horizontal"
+		(property "Footprint" "Diode_SMD:D_0201_0603Metric"
 			(at 165.1 68.58 0)
 			(effects
@@
 			)
 		)
-		(property "Footprint" "Diode_THT:D_5KPW_P12.70mm_Horizontal"
+		(property "Footprint" "Diode_SMD:D_0201_0603Metric"
 			(at 165.1 80.01 0)
 			(effects
@@
 			)
 		)
-		(property "Footprint" "Diode_THT:D_5KPW_P12.70mm_Horizontal"
+		(property "Footprint" "Diode_SMD:D_0201_0603Metric"
 			(at 185.42 45.72 0)
 			(effects
@@
 			)
 		)
-		(property "Footprint" "Diode_THT:D_5KPW_P12.70mm_Horizontal"
+		(property "Footprint" "Diode_SMD:D_0201_0603Metric"
 			(at 165.1 102.87 0)
 			(effects
@@
 			)
 		)
-		(property "Footprint" "Diode_THT:D_5KPW_P12.70mm_Horizontal"
+		(property "Footprint" "Diode_SMD:D_0201_0603Metric"
 			(at 185.42 102.87 0)
 			(effects
@@
 			)
 		)
-		(property "Footprint" "Diode_THT:D_5KPW_P12.70mm_Horizontal"
+		(property "Footprint" "Diode_SMD:D_0201_0603Metric"
 			(at 205.74 45.72 0)
 			(effects
@@
 			)
 		)
-		(property "Footprint" "Diode_THT:D_5KPW_P12.70mm_Horizontal"
+		(property "Footprint" "Diode_SMD:D_0201_0603Metric"
 			(at 165.1 45.72 0)
 			(effects
@@
 			)
 		)
-		(property "Footprint" "Diode_THT:D_5KPW_P12.70mm_Horizontal"
+		(property "Footprint" "Diode_SMD:D_0201_0603Metric"
 			(at 165.1 91.44 0)
 			(effects
@@
 			)
 		)
-		(property "Footprint" "Capacitor_THT:CP_Axial_L10.0mm_D4.5mm_P15.00mm_Horizontal"
+		(property "Footprint" "Capacitor_SMD:CP_Elec_3x5.3"
 			(at 121.92 124.46 0)
 			(effects
@@
 			)
 		)
-		(property "Footprint" "Diode_THT:D_5KPW_P12.70mm_Horizontal"
+		(property "Footprint" "Diode_SMD:D_0201_0603Metric"
 			(at 165.1 57.15 0)
 			(effects
@@
 			)
 		)
-		(property "Footprint" "Capacitor_THT:CP_Axial_L10.0mm_D4.5mm_P15.00mm_Horizontal"
+		(property "Footprint" "Capacitor_SMD:C_0201_0603Metric"
 			(at 117.1448 107.95 0)
 			(effects
@@
 			)
 		)
-		(property "Footprint" "Diode_THT:D_5KPW_P12.70mm_Horizontal"
+		(property "Footprint" "Diode_SMD:D_0201_0603Metric"
 			(at 185.42 91.44 0)
 			(effects
@@
 			)
 		)
-		(property "Footprint" "Capacitor_THT:CP_Axial_L10.0mm_D4.5mm_P15.00mm_Horizontal"
+		(property "Footprint" "Capacitor_SMD:C_0201_0603Metric"
 			(at 112.7252 132.08 0)
 			(effects
@@
 			)
 		)
-		(property "Footprint" "Diode_THT:D_5KPW_P12.70mm_Horizontal"
+		(property "Footprint" "Diode_SMD:D_0201_0603Metric"
 			(at 185.42 68.58 0)
 			(effects
@@
 			)
 		)
-		(property "Footprint" "Diode_THT:D_5KPW_P12.70mm_Horizontal"
+		(property "Footprint" "Diode_SMD:D_0201_0603Metric"
 			(at 205.74 57.15 0)
 			(effects
@@
 			)
 		)
-		(property "Footprint" "Diode_THT:D_5KPW_P12.70mm_Horizontal"
+		(property "Footprint" "Diode_SMD:D_0201_0603Metric"
 			(at 185.42 57.15 0)
 			(effects
@@
 			)
 		)
-		(property "Footprint" "Diode_THT:D_5KPW_P12.70mm_Horizontal"
+		(property "Footprint" "Diode_SMD:D_0201_0603Metric"
 			(at 185.42 80.01 0)
 			(effects

Commit message: fix: switch key switches for low profile
Parts:
- SW1, SW10, SW11, SW12, SW13, SW14, SW15, SW16, SW17, SW18, SW2, SW3, SW4, SW5, SW6, SW7, SW8, SW9: footprint PCM_Switch_Keyboard_Cherry_MX:SW_Cherry_MX_PCB -> 1 key-switches.pretty:SW_MX_LowProfile_THT
Changed lines of the file:
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@@
 			)
 		)
-		(property "Footprint" "PCM_Switch_Keyboard_Cherry_MX:SW_Cherry_MX_PCB"
+		(property "Footprint" "1 key-switches.pretty:SW_MX_LowProfile_THT"
 			(at 157.48 82.55 0)
 			(effects
@@
 			)
 		)
-		(property "Footprint" "PCM_Switch_Keyboard_Cherry_MX:SW_Cherry_MX_PCB"
+		(property "Footprint" "1 key-switches.pretty:SW_MX_LowProfile_THT"
 			(at 177.8 59.69 0)
 			(effects
@@
 			)
 		)
-		(property "Footprint" "PCM_Switch_Keyboard_Cherry_MX:SW_Cherry_MX_PCB"
+		(property "Footprint" "1 key-switches.pretty:SW_MX_LowProfile_THT"
 			(at 198.12 93.98 0)
 			(effects
@@
 			)
 		)
-		(property "Footprint" "PCM_Switch_Keyboard_Cherry_MX:SW_Cherry_MX_PCB"
+		(property "Footprint" "1 key-switches.pretty:SW_MX_LowProfile_THT"
 			(at 177.8 93.98 0)
 			(effects
@@
 			)
 		)
-		(property "Footprint" "PCM_Switch_Keyboard_Cherry_MX:SW_Cherry_MX_PCB"
+		(property "Footprint" "1 key-switches.pretty:SW_MX_LowProfile_THT"
 			(at 198.12 71.12 0)
 			(effects
@@
 			)
 		)
-		(property "Footprint" "PCM_Switch_Keyboard_Cherry_MX:SW_Cherry_MX_PCB"
+		(property "Footprint" "1 key-switches.pretty:SW_MX_LowProfile_THT"
 			(at 177.8 71.12 0)
 			(effects
@@
 			)
 		)
-		(property "Footprint" "PCM_Switch_Keyboard_Cherry_MX:SW_Cherry_MX_PCB"
+		(property "Footprint" "1 key-switches.pretty:SW_MX_LowProfile_THT"
 			(at 157.48 36.83 0)
 			(effects
@@
 			)
 		)
-		(property "Footprint" "PCM_Switch_Keyboard_Cherry_MX:SW_Cherry_MX_PCB"
+		(property "Footprint" "1 key-switches.pretty:SW_MX_LowProfile_THT"
 			(at 177.8 48.26 0)
 			(effects
@@
 			)
 		)
-		(property "Footprint" "PCM_Switch_Keyboard_Cherry_MX:SW_Cherry_MX_PCB"
+		(property "Footprint" "1 key-switches.pretty:SW_MX_LowProfile_THT"
 			(at 198.12 59.69 0)
 			(effects
@@
 			)
 		)
-		(property "Footprint" "PCM_Switch_Keyboard_Cherry_MX:SW_Cherry_MX_PCB"
+		(property "Footprint" "1 key-switches.pretty:SW_MX_LowProfile_THT"
 			(at 177.8 82.55 0)
 			(effects
@@
 			)
 		)
-		(property "Footprint" "PCM_Switch_Keyboard_Cherry_MX:SW_Cherry_MX_PCB"
+		(property "Footprint" "1 key-switches.pretty:SW_MX_LowProfile_THT"
 			(at 177.8 36.83 0)
 			(effects
@@
 			)
 		)
-		(property "Footprint" "PCM_Switch_Keyboard_Cherry_MX:SW_Cherry_MX_PCB"
+		(property "Footprint" "1 key-switches.pretty:SW_MX_LowProfile_THT"
 			(at 198.12 82.55 0)
 			(effects
@@
 			)
 		)
-		(property "Footprint" "PCM_Switch_Keyboard_Cherry_MX:SW_Cherry_MX_PCB"
+		(property "Footprint" "1 key-switches.pretty:SW_MX_LowProfile_THT"
 			(at 157.48 71.12 0)
 			(effects
@@
 			)
 		)
-		(property "Footprint" "PCM_Switch_Keyboard_Cherry_MX:SW_Cherry_MX_PCB"
+		(property "Footprint" "1 key-switches.pretty:SW_MX_LowProfile_THT"
 			(at 157.48 93.98 0)
 			(effects
@@
 			)
 		)
-		(property "Footprint" "PCM_Switch_Keyboard_Cherry_MX:SW_Cherry_MX_PCB"
+		(property "Footprint" "1 key-switches.pretty:SW_MX_LowProfile_THT"
 			(at 157.48 48.26 0)
 			(effects
@@
 			)
 		)
-		(property "Footprint" "PCM_Switch_Keyboard_Cherry_MX:SW_Cherry_MX_PCB"
+		(property "Footprint" "1 key-switches.pretty:SW_MX_LowProfile_THT"
 			(at 157.48 59.69 0)
 			(effects
@@
 			)
 		)
-		(property "Footprint" "PCM_Switch_Keyboard_Cherry_MX:SW_Cherry_MX_PCB"
+		(property "Footprint" "1 key-switches.pretty:SW_MX_LowProfile_THT"
 			(at 198.12 36.83 0)
 			(effects
@@
 			)
 		)
-		(property "Footprint" "PCM_Switch_Keyboard_Cherry_MX:SW_Cherry_MX_PCB"
+		(property "Footprint" "1 key-switches.pretty:SW_MX_LowProfile_THT"
 			(at 198.12 48.26 0)
 			(effects

Commit message: feat: routing
Parts:
- C1, C2, C3, C4, IC1, LS1, R3: now not fitted

Commit message: wip: backlight
Parts:
- added C5: 220 nF, Capacitor_THT:C_Disc_D3.0mm_W2.0mm_P2.50mm, symbol PCM_SL_Devices:Capacitor_NP
- added C6, C7: 1uF, Capacitor_SMD:C_0201_0603Metric, symbol Device:C
- added D20: MBR0540, Diode_SMD:D_SOD-123, symbol Diode:MBR0540
- added J2: TL040WVS03-H1263A, Connector_FFC-FPC:Hirose_FH12-40S-0.5SH_1x40-1MP_P0.50mm_Horizontal, symbol PiPhone Symbols:TL040WVS03-H1263A
- added J3: Conn_01x15_MountingPin, Connector_FFC-FPC:Molex_200528-0150_1x15-1MP_P1.00mm_Horizontal, symbol Connector_Generic_MountingPin:Conn_01x15_MountingPin
- added L1: 22uH, Inductor_SMD:L_6.3x6.3_H3, symbol Device:L
- added R1: 5, Resistor_SMD:R_0201_0603Metric, symbol Device:R
- added U1: ~, Package_DFN_QFN:QFN-48-1EP_6x6mm_P0.4mm_EP4.2x4.2mm, symbol PiPhone Symbols:ICN6211
- added U2: TPS61165DRV, Package_SON:WSON-6-1EP_2x2mm_P0.65mm_EP1x1.6mm, symbol Driver_LED:TPS61165DRV
- R3: footprint Diode_SMD:D_0201_0603Metric -> Resistor_SMD:R_0201_0603Metric
Connections:
- net +3V3: now also U1.24 (VDD2)
- net +5V: now also C6.2, L1.1, U2.6 (VIN)
- net GND: now also C5.1, C6.1, C7.1, J2.34 (GND), J2.4 (GND), J2.40 (GND), R1.2, U1.8 (TEST), U2.3 (GND), U2.7 (GND)
- net GPIO12/PWM0: now also U2.5 (CTRL)
- net GPIO24: now also J2.6 (RESET)
- net GPIO25: now also U1.11 (EN)
- net GPIO2/SDA1: now also J2.9 (SDA)
- net GPIO3/SCL1: now also J2.10 (SCK)
- net GPIO4/GPCLK0: now also J2.11 (CS)
- new net: C7.2, D20.1 (K), J2.1 (LED_A)
- new net: J2.12 (PCLK), U1.25 (PCLK)
- new net: J2.13 (DE), U1.28 (DATA_EN)
- new net: J2.14 (VSYNC), U1.27 (VSYNC)
- new net: J2.15 (HSYNC), U1.26 (HSYNC)
- new net: J2.16 (DB0), U1.7 (DATA23)
- new net: J2.17 (DB1), U1.6 (DATA22)
- new net: J2.18 (DB2), U1.5 (DATA21)
- new net: J2.19 (DB3), U1.4 (DATA20)
- new net: J2.2 (LED_K1), J2.3 (LED_K2), R1.1, U2.1 (FB)
- new net: J2.20 (DB4), U1.2 (DATA19)
- new net: J2.21 (DB5), U1.1 (DATA18)
- new net: J2.22 (DB6), U1.46 (DATA15)
- new net: J2.23 (DB7), U1.45 (DATA14)
- new net: J2.24 (DB8), U1.44 (DATA13)
- new net: J2.25 (DB9), U1.43 (DATA12)
- new net: J2.26 (DB10), U1.42 (DATA11)
- new net: J2.27 (DB11), U1.41 (DATA10)
- new net: J2.28 (DB12), U1.37 (DATA7)
- new net: J2.29 (DB13), U1.36 (DATA6)
- new net: J2.30 (DB14), U1.34 (DATA5)
- new net: J2.31 (DB15), U1.33 (DATA4)
- new net: J2.32 (DB16), U1.32 (DATA3)
- new net: J2.33 (DB17), U1.31 (DATA2)
- new net: J2.5 (VCI), U1.3 (VDD3)
- new net: J3.12 (Pin_12), U1.10 (SDA)
- new net: J3.14 (Pin_14), U1.12 (VDD1)
- new net: J3.9 (Pin_9), U1.14 (DA0P)
- new net: J3.8 (Pin_8), U1.15 (DA0N)
- new net: J3.3 (Pin_3), U1.16 (DA1P)
- new net: J3.2 (Pin_2), U1.17 (DA1N)
- new net: J3.6 (Pin_6), U1.18 (DACP)
- new net: J3.5 (Pin_5), U1.19 (DACN)
- new net: J3.1 (Pin_1), U1.35 (GND)
- new net: J3.11 (Pin_11), U1.9 (SCL)
- new net: D20.2 (A), L1.2, U2.4 (SW)
- new net: C5.2, U2.2 (COMP)
- no-connect marks 0 -> 17
Other:
- note added: "Backlight"
- note added: "Converter Enable"
- note added: "Keyboard"
- note added: "RBG Reset"
- note added: "Screen SPI"
- note added: "These bottom two unconnected are power The top unconected are GND"
- note added: "Touch Pins (Unused?)"

Commit message: feat: screen
Parts:
- removed C1: 100uf, Capacitor_SMD:CP_Elec_3x5.3, symbol Device:C_Polarized_US
- removed C2: 100uf, Capacitor_SMD:C_0201_0603Metric, symbol Device:C
- removed C3: 100nf, Capacitor_SMD:C_0201_0603Metric, symbol Device:C
- removed C4: 1000uf, Capacitor_SMD:CP_Elec_3x5.3, symbol Device:C_Polarized_US
- removed IC1: LM386M-1_NOPB, LM386M-1_NOBP:SOIC127P600X175-8N, symbol LM386M:LM386M-1_NOPB
- removed LS1: Speaker, Buzzer_Beeper:Speaker_CUI_CMR-1206S-67, symbol Device:Speaker
- removed R3: 10k, Resistor_SMD:R_0201_0603Metric, symbol Device:R
- C5: footprint Capacitor_THT:C_Disc_D3.0mm_W2.0mm_P2.50mm -> Capacitor_SMD:C_0201_0603Metric

Commit message: doc: document resistor values
Other:
- note added: "0.2v comes from the circuit docs"
- note added: "All of these other values in capacitors etc are from example and should be in a decent range"

Commit message: feat: protect backlight led
Parts:
- added R2: 320, Resistor_SMD:R_0201_0603Metric, symbol Device:R
Connections:
- net at C7.2, D20.1 (K): now also R2.1; no longer J2.1 (LED_A)
- new net: J2.1 (LED_A), R2.2
Changed lines of the file:
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@@
 	(wire
 		(pts
+			(xy 524.51 142.24) (xy 529.59 142.24)
+		)
+		(stroke
+			(width 0)
+			(type default)
+		)
+	)
+	(wire
+		(pts
 			(xy 165.1 95.25) (xy 185.42 95.25)
 		)
@@
 	(wire
 		(pts
-			(xy 516.89 142.24) (xy 529.59 142.24)
-		)
-		(stroke
-			(width 0)
-			(type default)
-		)
-	)
-	(wire
-		(pts
 			(xy 433.07 91.44) (xy 433.07 105.41)
 		)
@@
 	(wire
 		(pts
-			(xy 471.17 138.43) (xy 472.44 138.43)
+			(xy 464.82 138.43) (xy 472.44 138.43)
 		)
 		(stroke
@@
 	)
 	(symbol
+		(lib_id "Device:R")
+		(at 520.7 142.24 90)
+		(unit 1)
+		(exclude_from_sim no)
+		(in_bom yes)
+		(on_board yes)
+		(dnp no)
+		(fields_autoplaced yes)
+		(property "Reference" "R2"
+			(at 520.7 135.89 90)
+			(effects
+				(font
+					(size 1.27 1.27)
+				)
+			)
+		)
+		(property "Value" "320"
+			(at 520.7 138.43 90)
+			(effects
+				(font
+					(size 1.27 1.27)
+				)
+			)
+		)
+		(property "Footprint" "Resistor_SMD:R_0201_0603Metric"
+			(at 520.7 144.018 90)
+			(effects
+				(font
+					(size 1.27 1.27)
+				)
+				(hide yes)
+			)
+		)
+		(property "Datasheet" "~"
+			(at 520.7 142.24 0)
+			(effects
+				(font
+					(size 1.27 1.27)
+				)
+				(hide yes)
+			)
+		)
+		(property "Description" "Resistor"
+			(at 520.7 142.24 0)
+			(effects
+				(font
+					(size 1.27 1.27)
+				)
+				(hide yes)
+			)
+		)
+		(pin "2"
+		)
+		(pin "1"
+		)
+		(instances
+			(project ""
+				(path "/e63e39d7-6ac0-4ffd-8aa3-1841a4541b55"
+					(reference "R2")
+					(unit 1)
+				)
+			)
+		)
+	)
+	(symbol
 		(lib_id "Device:D")
 		(at 205.74 68.58 90)
@@
 	(symbol
 		(lib_id "power:+5V")
-		(at 471.17 138.43 90)
+		(at 464.82 138.43 90)
 		(unit 1)
 		(exclude_from_sim no)
@@
 		(dnp no)
 		(property "Reference" "#PWR019"
-			(at 474.98 138.43 0)
+			(at 468.63 138.43 0)
 			(effects
 				(font
@@
 		)
 		(property "Value" "+5V"
-			(at 466.8456 138.0617 0)
+			(at 460.4956 138.0617 0)
 			(effects
 				(font
@@
 		)
 		(property "Footprint" ""
-			(at 471.17 138.43 0)
+			(at 464.82 138.43 0)
 			(effects
 				(font
@@
 		)
 		(property "Datasheet" ""
-			(at 471.17 138.43 0)
+			(at 464.82 138.43 0)
 			(effects
 				(font
@@
 		)
 		(property "Description" "Power symbol creates a global label with name \"+5V\""
-			(at 471.17 138.43 0)
+			(at 464.82 138.43 0)
 			(effects
 				(font

Commit message: docs: protect backlight led note
Other:
- note added: "R2 is protecting the LED 12.8v 40mA"
Changed lines of the file:
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@@
 		)
 	)
+	(text "R2 is protecting the LED\n12.8v 40mA"
+		(exclude_from_sim no)
+		(at 540.004 147.32 0)
+		(effects
+			(font
+				(size 1.27 1.27)
+			)
+		)
+	)
 	(text "Keyboard"
 		(exclude_from_sim no)
@@
 		)
 		(property "Value" "+3V3"
-			(at 433.8256 122.8217 0)
+			(at 433.832 123.19 0)
 			(effects
 				(font
